Commit message: Replace project snapshot with two-way USBL EKF fusion and updated navigation results
Publish the complete 119-file local project snapshot, including acoustic position fusion, regression tests, README, measured trajectories and regenerated 2D/3D figures.

File: baseline_robot_description/urdf/base.urdf (robot description, URDF)
Before this commit: robot baseline_robot, 15 links, 14 joints
Links:
- added link acoustic_transponder
Joints:
- added joint acoustic_transponder_joint: type fixed, parent base_link, child acoustic_transponder, origin xyz=0.0 0.0 0.0 rpy=3.141592653589793 0.0 0.0
